File: experimental/splitterbox/eagle/eagle/SplitterBoxRevC.brd (EAGLE design)
At the start: 86.4 x 76.2 mm, 73 parts, among them IC1 ATMEGA328P_PDIP, IC101 FT232RL, IC2 MAX233, IC201 FT232RL, IC301 FT232RL, IC401 FT232RL, IC501 FT232RL, IC601 FT232RL

Commit message: Updates
Parts:
- removed R3: 10K, SparkFun-Passives:AXIAL-0.4
- added LOGO1: OSHW-LOGOS, SparkFun-Aesthetics:OSHW-LOGO-S
- moved C401 2.54 mm to (72.4, 64.8), turned to 180 degrees
Connections:
- removed net N$8: MODE.1, MODE.2, R3.P$2
- net MOSI: now also MODE.1, MODE.2; no longer R3.P$1
Routing:
- net MOSI: track 18.1 -> 45.9 mm
- net N$8: track 14.1 -> 0.00 mm
- net N$6: track 12.5 -> 15.1 mm
Other:
- board text added: "MODE"
- board text added: "Rev C 08/2016"
- board text added: "Simulator Splitter Box"
- board text removed: "Rev 1 09/2015"
- board text removed: "Splittter Box Functional Prototype"
