File: experimental/splitterbox/eagle/eagle/SplitterBoxRevC.sch (EAGLE design)
At the start: 73 parts, among them IC1 ATMEGA328P_PDIP, IC101 FT232RL, IC2 MAX233, IC201 FT232RL, IC301 FT232RL, IC401 FT232RL, IC501 FT232RL, IC601 FT232RL

Commit message: Updates
Parts:
- removed R3: 10K, SparkFun-Passives:RESISTORPTH-1/4W
- added LOGO1: OSHW-LOGOS, SparkFun-Aesthetics:OSHW-LOGOS
Connections:
- removed net N$8: MODE.S, MODE.S1, R3.2
- net MOSI: now also MODE.S, MODE.S1; no longer R3.1
Other:
- moved on the sheet: C2, C3, C4, C5, C6, IC2P, L1, LED1, MODE, R2, TP1
