File: experimental/tvsboard/hardware/eagle/InterfaceTVSBoardRevB.brd (EAGLE design)
At the start: 33 x 52.1 mm, 30 parts, among them IC1 USB6B1, IC2 USB6B1, IC3 USB6B1, IC4 USB6B1, IC5 USB6B1, IC6 USB6B1

Commit message: Updates
Parts:
- removed IC1, IC2, IC3, IC4, IC5, IC6: USB6B1, st-microelectronics:SO08
- added D0, D1, D2, D3, D4, D5, D6, D7, D8, D9, DE, DT: SA5.0A, AIC_Custom:DO41_TVS_UNI
- added LOGO1: OSHW-LOGOS, SparkFun-Aesthetics:OSHW-LOGO-S
Connections:
- removed net N$13: IC4.3, S7.3
- removed net N$14: IC4.2, S8.3
- removed net N$15: IC5.3, S9.3
- removed net N$16: B9.3, IC5.6
- removed net N$18: IC6.3, SE.3
- removed net N$19: BE.3, IC6.6
- removed net N$20: B8.3, IC4.7
- removed net N$21: B7.3, IC4.6
- removed net N$22: IC6.2, ST.3
- removed net N$23: BT.3, IC6.7
- removed net N$24: IC5.2, S0.3
- removed net N$25: B0.3, IC5.7
- net GND: now also D0.ANODE, D1.ANODE, D2.ANODE, D3.ANODE, D4.ANODE, D5.ANODE, D6.ANODE, D7.ANODE, D8.ANODE, D9.ANODE, DE.ANODE, DT.ANODE; no longer IC1.4, IC1.5, IC2.4, IC2.5, IC3.4, IC3.5, IC4.4, IC4.5, IC5.4, IC5.5, IC6.4, IC6.5
- net N$1: now also B1.3, D1.CATHODE; no longer IC1.3
- net N$10: now also B0.3, D0.CATHODE, S0.3; no longer B5.3, IC3.6
- net N$11: now also BE.3, DE.CATHODE, SE.3; no longer IC3.2, S6.3
- net N$12: now also BT.3, DT.CATHODE, ST.3; no longer B6.3, IC3.7
- net N$2: now also B2.3, D2.CATHODE; no longer IC1.2
- net N$3: now also B3.3, D3.CATHODE, S3.3; no longer B1.3, IC1.6
- net N$4: now also B4.3, D4.CATHODE, S4.3; no longer B2.3, IC1.7
- net N$5: now also B5.3, D5.CATHODE, S5.3; no longer IC2.3, S3.3
- net N$6: now also B6.3, D6.CATHODE, S6.3; no longer B3.3, IC2.6
- net N$7: now also B7.3, D7.CATHODE, S7.3; no longer IC2.2, S4.3
- net N$8: now also B8.3, D8.CATHODE, S8.3; no longer B4.3, IC2.7
- net N$9: now also B9.3, D9.CATHODE, S9.3; no longer IC3.3, S5.3
- net VCC: no longer IC1.1, IC1.8, IC2.1, IC2.8, IC3.1, IC3.8, IC4.1, IC4.8, IC5.1, IC5.8, IC6.1, IC6.8
Routing:
- net VCC: track 153.6 -> 87.4 mm
- net N$12: track 5.27 -> 21.4 mm
- net N$6: track 5.27 -> 21.4 mm
- net N$10: track 5.86 -> 21.5 mm
- net N$8: track 5.86 -> 21.4 mm
- net N$3: track 6.39 -> 21.4 mm
- net N$4: track 6.89 -> 21.4 mm
- net N$18: track 12.9 -> 0.00 mm
- net N$14: track 12.9 -> 0.00 mm
- net N$22: track 11.4 -> 0.00 mm
- net N$13: track 11.1 -> 0.00 mm
- net N$24: track 10.9 -> 0.00 mm
- net N$15: track 10.9 -> 0.00 mm
- net N$11: track 10.8 -> 21.5 mm
- net N$7: track 10.9 -> 21.5 mm
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Other:
- board text added: "Rev B 08/2016"
- board text added: "Simulator Interface TVS Board"
- board text removed: "Interface TVS Board"
- board text removed: "Rev A 04/2016"
